File: jrdish_axis_controller/user_switches.kicad_sch (KiCad schematic)
At the start: 1 part, among them CN14 KF2EDGR-2.54-6P

Commit message: Near finished routing
Parts:
- added C72, C73, C74, C75: 100nF, PCM_JLCPCB:C_0402, symbol PCM_JLCPCB-Capacitors:0402,100nF
- added D12, D13, D14, D15: TPESD0402G05V, MyParts:D0402-BI, symbol MyParts:TPESD0402G05V
- added R47, R49, R51, R53: 4.7kΩ, PCM_JLCPCB:R_0402, symbol PCM_JLCPCB-Resistors:0402,4.7kΩ
- added R48, R50, R52, R54: 100Ω, PCM_JLCPCB:R_0402, symbol PCM_JLCPCB-Resistors:0402,100Ω
Connections:
- net USER_SW_1_MCU: now also C72.1, R48.2
- net USER_SW_2_MCU: now also C73.1, R50.2
- net USER_SW_3_MCU: now also C74.1, R52.2
- net USER_SW_4_MCU: now also C75.1, R54.2
- net USER_SW_1: now reaches CN14.1
- net USER_SW_1: now also D12.1 (K), R47.2, R48.1
- net GND: now reaches CN14.2
- net GND: now also CN14.5, C72.2, C73.2, C74.2, C75.2, D12.2 (A), D13.2 (A), D14.2 (A), D15.2 (A)
- net USER_SW_2: now reaches CN14.3
- net USER_SW_2: now also D13.1 (K), R49.2, R50.1
- net USER_SW_3: now reaches CN14.4
- net USER_SW_3: now also D14.1 (K), R51.2, R52.1
- net USER_SW_4: now reaches CN14.6
- net USER_SW_4: now also D15.1 (K), R53.2, R54.1
- new net 3V3: R47.1, R49.1, R51.1, R53.1
Other:
- note added: "Gnd"
- note added: "Inputs to four switches for general use. It is envisioned using 2 toggle switches to allow manually moving the dish."
- note added: "USER_SW_1"
- note added: "USER_SW_2"
- note added: "USER_SW_3"
- note added: "USER_SW_4"
- moved on the sheet: CN14

Commit message: Layout complete
Changed lines of the file:
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@@
 	)
 	(symbol
+		(lib_name "TPESD0402G05V_2")
 		(lib_id "MyParts:TPESD0402G05V")
 		(at 128.27 85.09 270)
@@
 			)
 		)
-		(property "Datasheet" ""
+		(property "Datasheet" "https://www.lcsc.com/datasheet/C558615.pdf?spm=wm.sxq.inf.ggs___wm.ssy.bg.0.xh&lcsc_vid=FFBaV1wHQFldUVICFgBfBVJTQVJWXgBfEQRYBAFQE1YxVlNRQFVXU1JRQVReUTsOAxUeFF5JWBYZEEoKFBINSQcJGk4eFQsCAgIaSgADAwAHC0slRldcU1ZUWQkaCgg%3D"
 			(at 128.27 85.09 0)
 			(hide yes)
@@
 			)
 		)
-		(property "Description" ""
+		(property "Description" "5VWM 40VC 0402"
 			(at 128.27 85.09 0)
 			(hide yes)
@@
 	)
 	(symbol
+		(lib_name "TPESD0402G05V_3")
 		(lib_id "MyParts:TPESD0402G05V")
 		(at 128.27 115.57 270)
@@
 			)
 		)
-		(property "Datasheet" ""
+		(property "Datasheet" "https://www.lcsc.com/datasheet/C558615.pdf?spm=wm.sxq.inf.ggs___wm.ssy.bg.0.xh&lcsc_vid=FFBaV1wHQFldUVICFgBfBVJTQVJWXgBfEQRYBAFQE1YxVlNRQFVXU1JRQVReUTsOAxUeFF5JWBYZEEoKFBINSQcJGk4eFQsCAgIaSgADAwAHC0slRldcU1ZUWQkaCgg%3D"
 			(at 128.27 115.57 0)
 			(hide yes)
@@
 			)
 		)
-		(property "Description" ""
+		(property "Description" "5VWM 40VC 0402"
 			(at 128.27 115.57 0)
 			(hide yes)
@@
 			)
 		)
-		(property "Datasheet" ""
+		(property "Datasheet" "https://www.lcsc.com/datasheet/C558615.pdf?spm=wm.sxq.inf.ggs___wm.ssy.bg.0.xh&lcsc_vid=FFBaV1wHQFldUVICFgBfBVJTQVJWXgBfEQRYBAFQE1YxVlNRQFVXU1JRQVReUTsOAxUeFF5JWBYZEEoKFBINSQcJGk4eFQsCAgIaSgADAwAHC0slRldcU1ZUWQkaCgg%3D"
 			(at 129.54 147.32 0)
 			(hide yes)
@@
 			)
 		)
-		(property "Description" ""
+		(property "Description" "5VWM 40VC 0402"
 			(at 129.54 147.32 0)
 			(hide yes)
@@
 	)
 	(symbol
+		(lib_name "TPESD0402G05V_1")
 		(lib_id "MyParts:TPESD0402G05V")
 		(at 128.27 54.61 270)
@@
 			)
 		)
-		(property "Datasheet" ""
+		(property "Datasheet" "https://www.lcsc.com/datasheet/C558615.pdf?spm=wm.sxq.inf.ggs___wm.ssy.bg.0.xh&lcsc_vid=FFBaV1wHQFldUVICFgBfBVJTQVJWXgBfEQRYBAFQE1YxVlNRQFVXU1JRQVReUTsOAxUeFF5JWBYZEEoKFBINSQcJGk4eFQsCAgIaSgADAwAHC0slRldcU1ZUWQkaCgg%3D"
 			(at 128.27 54.61 0)
 			(hide yes)
@@
 			)
 		)
-		(property "Description" ""
+		(property "Description" "5VWM 40VC 0402"
 			(at 128.27 54.61 0)
 			(hide yes)

Commit message: Making refinements
Connections:
- removed net GND: C72.2, C73.2, C74.2, C75.2, CN14.2, CN14.5, D12.2 (A), D13.2 (A), D14.2 (A), D15.2 (A)
- new net: C73.2, D13.2 (A)
- new net: C75.2, D15.2 (A)
- new net: C74.2, D14.2 (A)
- new net: CN14.2, CN14.5
- new net: C72.2, D12.2 (A)
Other:
- company: (none) -> JRSeti
- title: (none) -> User Switches
Changed lines of the file:
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@@
 	(generator_version "10.0")
 	(paper "A4")
+	(title_block
+		(title "User Switches")
+		(date "2026-04-30")
+		(rev "1.0")
+		(company "JRSeti")
+	)
 	(text "USER_SW_2"
 		(exclude_from_sim no)

Commit message: Limit switches with mosfets
Connections:
- net GND: now reaches C73.2, D13.2 (A)
- net GND: now also C72.2, C74.2, C75.2, CN14.2, CN14.5, D12.2 (A), D14.2 (A), D15.2 (A)
Changed lines of the file:
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@@
 	)
 	(symbol
-		(lib_name "TPESD0402G05V_2")
 		(lib_id "MyParts:TPESD0402G05V")
 		(at 128.27 85.09 270)
@@
 	)
 	(symbol
-		(lib_name "TPESD0402G05V_3")
 		(lib_id "MyParts:TPESD0402G05V")
 		(at 128.27 115.57 270)
@@
 	)
 	(symbol
-		(lib_name "TPESD0402G05V_1")
 		(lib_id "MyParts:TPESD0402G05V")
 		(at 128.27 54.61 270)
