File: jrdish_axis_controller/gps_rs232.kicad_sch (KiCad schematic)
At the start: 11 parts, among them CN10 KF2EDGR-2.54-3P, CN9 KF2EDGR-2.54-2P, Q3 2N7002, U8 SP3232EEY-L/TR

Commit message: Continuing layout
Parts:
- renumbered C48 to C57, C49 to C58, C50 to C59, C52 to C60, C51 to C61, CN10 to CN5, CN9 to CN6, R30 to R29, R28 to R30
Changed lines of the file:
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@@
 		(dnp no)
 		(fields_autoplaced yes)
-		(property "Reference" "#PWR050"
+		(property "Reference" "#PWR052"
 			(at 168.91 134.62 0)
 			(hide yes)
@@
 			(project "jrdish_axis_controller"
 				(path "/10d7c3e5-be4d-4306-a59e-500b86bd141f/005a8950-9739-403f-9896-26bcf992d086"
-					(reference "#PWR050")
+					(reference "#PWR052")
 					(unit 1)
 				)
@@
 		(dnp no)
 		(fields_autoplaced yes)
-		(property "Reference" "C49"
+		(property "Reference" "C58"
 			(at 125.73 102.87 90)
 			(show_name no)
@@
 			(project "jrdish_axis_controller"
 				(path "/10d7c3e5-be4d-4306-a59e-500b86bd141f/005a8950-9739-403f-9896-26bcf992d086"
-					(reference "C49")
+					(reference "C58")
 					(unit 1)
 				)
@@
 		(in_pos_files yes)
 		(dnp no)
-		(property "Reference" "CN9"
+		(property "Reference" "CN6"
 			(at 123.952 59.944 0)
 			(show_name no)
@@
 			(project "jrdish_axis_controller"
 				(path "/10d7c3e5-be4d-4306-a59e-500b86bd141f/005a8950-9739-403f-9896-26bcf992d086"
-					(reference "CN9")
+					(reference "CN6")
 					(unit 1)
 				)
@@
 		(dnp no)
 		(fields_autoplaced yes)
-		(property "Reference" "#PWR052"
+		(property "Reference" "#PWR051"
 			(at 181.61 129.54 0)
 			(hide yes)
@@
 			(project "jrdish_axis_controller"
 				(path "/10d7c3e5-be4d-4306-a59e-500b86bd141f/005a8950-9739-403f-9896-26bcf992d086"
-					(reference "#PWR052")
+					(reference "#PWR051")
 					(unit 1)
 				)
@@
 		(dnp no)
 		(fields_autoplaced yes)
-		(property "Reference" "#PWR047"
+		(property "Reference" "#PWR049"
 			(at 144.78 76.2 0)
 			(hide yes)
@@
 			(project "jrdish_axis_controller"
 				(path "/10d7c3e5-be4d-4306-a59e-500b86bd141f/005a8950-9739-403f-9896-26bcf992d086"
-					(reference "#PWR047")
+					(reference "#PWR049")
 					(unit 1)
 				)
@@
 		(in_pos_files yes)
 		(dnp no)
-		(property "Reference" "C50"
+		(property "Reference" "C59"
 			(at 108.458 117.094 90)
 			(show_name no)
@@
 			(project "jrdish_axis_controller"
 				(path "/10d7c3e5-be4d-4306-a59e-500b86bd141f/005a8950-9739-403f-9896-26bcf992d086"
-					(reference "C50")
+					(reference "C59")
 					(unit 1)
 				)
@@
 		(in_pos_files yes)
 		(dnp no)
-		(property "Reference" "CN10"
+		(property "Reference" "CN5"
 			(at 185.674 113.03 0)
 			(show_name no)
@@
 			(project "jrdish_axis_controller"
 				(path "/10d7c3e5-be4d-4306-a59e-500b86bd141f/005a8950-9739-403f-9896-26bcf992d086"
-					(reference "CN10")
+					(reference "CN5")
 					(unit 1)
 				)
@@
 		(dnp no)
 		(fields_autoplaced yes)
-		(property "Reference" "R30"
+		(property "Reference" "R29"
 			(at 147.32 52.0699 0)
 			(show_name no)
@@
 			(project "jrdish_axis_controller"
 				(path "/10d7c3e5-be4d-4306-a59e-500b86bd141f/005a8950-9739-403f-9896-26bcf992d086"
-					(reference "R30")
+					(reference "R29")
 					(unit 1)
 				)
@@
 		(dnp no)
 		(fields_autoplaced yes)
-		(property "Reference" "#PWR049"
+		(property "Reference" "#PWR053"
 			(at 129.54 137.16 0)
 			(hide yes)
@@
 			(project "jrdish_axis_controller"
 				(path "/10d7c3e5-be4d-4306-a59e-500b86bd141f/005a8950-9739-403f-9896-26bcf992d086"
-					(reference "#PWR049")
+					(reference "#PWR053")
 					(unit 1)
 				)
@@
 		(dnp no)
 		(fields_autoplaced yes)
-		(property "Reference" "#PWR046"
+		(property "Reference" "#PWR048"
 			(at 128.27 73.66 0)
 			(hide yes)
@@
 			(project "jrdish_axis_controller"
 				(path "/10d7c3e5-be4d-4306-a59e-500b86bd141f/005a8950-9739-403f-9896-26bcf992d086"
-					(reference "#PWR046")
+					(reference "#PWR048")
 					(unit 1)
 				)
@@
 		(dnp no)
 		(fields_autoplaced yes)
-		(property "Reference" "R28"
+		(property "Reference" "R30"
 			(at 132.08 59.69 90)
 			(show_name no)
@@
 			(project "jrdish_axis_controller"
 				(path "/10d7c3e5-be4d-4306-a59e-500b86bd141f/005a8950-9739-403f-9896-26bcf992d086"
-					(reference "R28")
+					(reference "R30")
 					(unit 1)
 				)
@@
 		(in_pos_files yes)
 		(dnp no)
-		(property "Reference" "C51"
+		(property "Reference" "C61"
 			(at 108.712 126.492 90)
 			(show_name no)
@@
 			(project "jrdish_axis_controller"
 				(path "/10d7c3e5-be4d-4306-a59e-500b86bd141f/005a8950-9739-403f-9896-26bcf992d086"
-					(reference "C51")
+					(reference "C61")
 					(unit 1)
 				)
@@
 		(dnp no)
 		(fields_autoplaced yes)
-		(property "Reference" "#PWR048"
+		(property "Reference" "#PWR054"
 			(at 109.22 139.7 0)
 			(hide yes)
@@
 			(project "jrdish_axis_controller"
 				(path "/10d7c3e5-be4d-4306-a59e-500b86bd141f/005a8950-9739-403f-9896-26bcf992d086"
-					(reference "#PWR048")
+					(reference "#PWR054")
 					(unit 1)
 				)
@@
 		(in_pos_files yes)
 		(dnp no)
-		(property "Reference" "C52"
+		(property "Reference" "C60"
 			(at 122.682 117.856 90)
 			(show_name no)
@@
 			(project "jrdish_axis_controller"
 				(path "/10d7c3e5-be4d-4306-a59e-500b86bd141f/005a8950-9739-403f-9896-26bcf992d086"
-					(reference "C52")
+					(reference "C60")
 					(unit 1)
 				)
@@
 		(dnp no)
 		(fields_autoplaced yes)
-		(property "Reference" "#PWR051"
+		(property "Reference" "#PWR050"
 			(at 168.91 114.3 0)
 			(hide yes)
@@
 			(project "jrdish_axis_controller"
 				(path "/10d7c3e5-be4d-4306-a59e-500b86bd141f/005a8950-9739-403f-9896-26bcf992d086"
-					(reference "#PWR051")
+					(reference "#PWR050")
 					(unit 1)
 				)
@@
 		(in_pos_files yes)
 		(dnp no)
-		(property "Reference" "C48"
+		(property "Reference" "C57"
 			(at 164.592 105.1559 0)
 			(show_name no)
@@
 			(project "jrdish_axis_controller"
 				(path "/10d7c3e5-be4d-4306-a59e-500b86bd141f/005a8950-9739-403f-9896-26bcf992d086"
-					(reference "C48")
+					(reference "C57")
 					(unit 1)
 				)

Commit message: RS485 isolated areas in place
Parts:
- renumbered C58 to C62, C57 to C63, C59 to C64, C60 to C65, C61 to C66, CN6 to CN10, CN5 to CN11, R29 to R31, R30 to R32
Connections:
- net 3V3: now also U8.16 (VCC)
- net GND: now also C63.2
Other:
- moved on the sheet: C63
Changed lines of the file:
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@@
 	(text "RS232"
 		(exclude_from_sim no)
-		(at 110.998 97.536 0)
+		(at 109.22 97.282 0)
 		(effects
 			(font
@@
 	)
 	(junction
+		(at 162.56 111.76)
+		(diameter 0)
+		(color 0 0 0 0)
+	)
+	(junction
 		(at 109.22 124.46)
 		(diameter 0)
@@
 	)
 	(junction
+		(at 172.72 113.03)
+		(diameter 0)
+		(color 0 0 0 0)
+	)
+	(junction
 		(at 144.78 57.15)
 		(diameter 0)
@@
 	(wire
 		(pts
+			(xy 162.56 111.76) (xy 163.83 111.76)
+		)
+		(stroke
+			(width 0)
+			(type default)
+		)
+	)
+	(wire
+		(pts
 			(xy 161.29 119.38) (xy 182.88 119.38)
 		)
@@
 	(wire
 		(pts
-			(xy 161.29 114.3) (xy 162.56 114.3)
+			(xy 161.29 114.3) (xy 172.72 114.3)
 		)
 		(stroke
@@
 	(wire
 		(pts
-			(xy 162.56 110.49) (xy 162.56 111.76)
+			(xy 127 63.5) (xy 128.27 63.5)
 		)
 		(stroke
@@
 	(wire
 		(pts
-			(xy 127 63.5) (xy 128.27 63.5)
+			(xy 172.72 111.76) (xy 172.72 113.03)
 		)
 		(stroke
@@
 	(wire
 		(pts
-			(xy 162.56 101.6) (xy 162.56 102.87)
+			(xy 144.78 46.99) (xy 143.51 46.99)
 		)
 		(stroke
@@
 	(wire
 		(pts
-			(xy 144.78 46.99) (xy 143.51 46.99)
+			(xy 118.11 114.3) (xy 130.81 114.3)
 		)
 		(stroke
@@
 	(wire
 		(pts
-			(xy 118.11 114.3) (xy 130.81 114.3)
+			(xy 181.61 121.92) (xy 181.61 123.19)
 		)
 		(stroke
@@
 	(wire
 		(pts
-			(xy 181.61 121.92) (xy 181.61 123.19)
+			(xy 110.49 114.3) (xy 109.22 114.3)
 		)
 		(stroke
@@
 	(wire
 		(pts
-			(xy 163.83 101.6) (xy 162.56 101.6)
+			(xy 161.29 116.84) (xy 182.88 116.84)
 		)
 		(stroke
@@
 	(wire
 		(pts
-			(xy 110.49 114.3) (xy 109.22 114.3)
+			(xy 172.72 113.03) (xy 172.72 114.3)
 		)
 		(stroke
@@
 	(wire
 		(pts
-			(xy 161.29 116.84) (xy 182.88 116.84)
+			(xy 109.22 114.3) (xy 109.22 124.46)
 		)
 		(stroke
@@
 	(wire
 		(pts
-			(xy 109.22 114.3) (xy 109.22 124.46)
+			(xy 162.56 109.22) (xy 162.56 111.76)
 		)
 		(stroke
@@
 	(wire
 		(pts
+			(xy 171.45 111.76) (xy 172.72 111.76)
+		)
+		(stroke
+			(width 0)
+			(type default)
+		)
+	)
+	(wire
+		(pts
 			(xy 120.65 119.38) (xy 120.65 121.92)
 		)
@@
 	(wire
 		(pts
+			(xy 172.72 113.03) (xy 176.53 113.03)
+		)
+		(stroke
+			(width 0)
+			(type default)
+		)
+	)
+	(wire
+		(pts
 			(xy 127 66.04) (xy 128.27 66.04)
 		)
@@
 	(global_label "3V3"
 		(shape input)
-		(at 163.83 101.6 0)
+		(at 162.56 109.22 90)
 		(fields_autoplaced yes)
 		(effects
@@
 		)
 		(property "Intersheetrefs" "${INTERSHEET_REFS}"
-			(at 170.3228 101.6 0)
+			(at 162.56 102.7272 90)
 			(hide yes)
 			(show_name no)
@@
 		(dnp no)
 		(fields_autoplaced yes)
-		(property "Reference" "C58"
+		(property "Reference" "C62"
 			(at 125.73 102.87 90)
 			(show_name no)
@@
 			(project "jrdish_axis_controller"
 				(path "/10d7c3e5-be4d-4306-a59e-500b86bd141f/005a8950-9739-403f-9896-26bcf992d086"
-					(reference "C58")
+					(reference "C62")
 					(unit 1)
 				)
@@
 		(in_pos_files yes)
 		(dnp no)
-		(property "Reference" "CN6"
+		(property "Reference" "CN10"
 			(at 123.952 59.944 0)
 			(show_name no)
@@
 			(project "jrdish_axis_controller"
 				(path "/10d7c3e5-be4d-4306-a59e-500b86bd141f/005a8950-9739-403f-9896-26bcf992d086"
-					(reference "CN6")
+					(reference "CN10")
 					(unit 1)
 				)
@@
 		(in_pos_files yes)
 		(dnp no)
-		(property "Reference" "C59"
+		(property "Reference" "C64"
 			(at 108.458 117.094 90)
 			(show_name no)
@@
 			(project "jrdish_axis_controller"
 				(path "/10d7c3e5-be4d-4306-a59e-500b86bd141f/005a8950-9739-403f-9896-26bcf992d086"
-					(reference "C59")
+					(reference "C64")
 					(unit 1)
 				)
@@
 		(in_pos_files yes)
 		(dnp no)
-		(property "Reference" "CN5"
+		(property "Reference" "CN11"
 			(at 185.674 113.03 0)
 			(show_name no)
@@
 			(project "jrdish_axis_controller"
 				(path "/10d7c3e5-be4d-4306-a59e-500b86bd141f/005a8950-9739-403f-9896-26bcf992d086"
-					(reference "CN5")
+					(reference "CN11")
 					(unit 1)
 				)
@@
 		(dnp no)
 		(fields_autoplaced yes)
-		(property "Reference" "R29"
+		(property "Reference" "R31"
 			(at 147.32 52.0699 0)
 			(show_name no)
@@
 			(project "jrdish_axis_controller"
 				(path "/10d7c3e5-be4d-4306-a59e-500b86bd141f/005a8950-9739-403f-9896-26bcf992d086"
-					(reference "R29")
+					(reference "R31")
 					(unit 1)
 				)
@@
 		(dnp no)
 		(fields_autoplaced yes)
-		(property "Reference" "R30"
+		(property "Reference" "R32"
 			(at 132.08 59.69 90)
 			(show_name no)
@@
 			(project "jrdish_axis_controller"
 				(path "/10d7c3e5-be4d-4306-a59e-500b86bd141f/005a8950-9739-403f-9896-26bcf992d086"
-					(reference "R30")
+					(reference "R32")
 					(unit 1)
 				)
@@
 		(in_pos_files yes)
 		(dnp no)
-		(property "Reference" "C61"
+		(property "Reference" "C66"
 			(at 108.712 126.492 90)
 			(show_name no)
@@
 			(project "jrdish_axis_controller"
 				(path "/10d7c3e5-be4d-4306-a59e-500b86bd141f/005a8950-9739-403f-9896-26bcf992d086"
-					(reference "C61")
+					(reference "C66")
 					(unit 1)
 				)
@@
 		(in_pos_files yes)
 		(dnp no)
-		(property "Reference" "C60"
+		(property "Reference" "C65"
 			(at 122.682 117.856 90)
 			(show_name no)
@@
 			(project "jrdish_axis_controller"
 				(path "/10d7c3e5-be4d-4306-a59e-500b86bd141f/005a8950-9739-403f-9896-26bcf992d086"
-					(reference "C60")
+					(reference "C65")
 					(unit 1)
 				)
@@
 	(symbol
 		(lib_id "power:GND")
-		(at 162.56 114.3 90)
+		(at 176.53 113.03 0)
 		(unit 1)
 		(body_style 1)
@@
 		(fields_autoplaced yes)
 		(property "Reference" "#PWR050"
-			(at 168.91 114.3 0)
+			(at 176.53 119.38 0)
 			(hide yes)
 			(show_name no)
@@
 		)
 		(property "Value" "GND"
-			(at 167.64 114.3 0)
+			(at 176.53 118.11 0)
 			(hide yes)
 			(show_name no)
@@
 		)
 		(property "Footprint" ""
-			(at 162.56 114.3 0)
+			(at 176.53 113.03 0)
 			(hide yes)
 			(show_name no)
@@
 		)
 		(property "Datasheet" ""
-			(at 162.56 114.3 0)
+			(at 176.53 113.03 0)
 			(hide yes)
 			(show_name no)
@@
 		)
 		(property "Description" "Power symbol creates a global label with name \"GND\" , ground"
-			(at 162.56 114.3 0)
+			(at 176.53 113.03 0)
 			(hide yes)
 			(show_name no)
@@
 	(symbol
 		(lib_id "PCM_JLCPCB-Capacitors:0402,100nF")
-		(at 162.56 106.68 0)
+		(at 167.64 111.76 90)
 		(unit 1)
 		(body_style 1)
@@
 		(in_pos_files yes)
 		(dnp no)
-		(property "Reference" "C57"
-			(at 164.592 105.1559 0)
+		(property "Reference" "C63"
+			(at 166.624 106.4259 90)
 			(show_name no)
 			(do_not_autoplace no)
@@
 					(size 1.27 1.27)
 				)
-				(justify left)
+				(justify right)
 			)
 		)
 		(property "Value" "100nF"
-			(at 164.592 107.696 0)
+			(at 166.624 108.204 90)
 			(show_name no)
 			(do_not_autoplace no)
@@
 					(size 0.8 0.8)
 				)
-				(justify left)
+				(justify right)
 			)
 		)
 		(property "Footprint" "PCM_JLCPCB:C_0402"
-			(at 160.782 106.68 90)
+			(at 167.64 113.538 90)
 			(hide yes)
 			(show_name no)
@@
 		)
 		(property "Datasheet" "https://www.lcsc.com/datasheet/lcsc_datasheet_2304140030_Samsung-Electro-Mechanics-CL05B104KO5NNNC_C1525.pdf"
-			(at 162.56 106.68 0)
+			(at 167.64 111.76 0)
 			(hide yes)
 			(show_name no)
@@
 		)
 		(property "Description" "16V 100nF X7R ±10% 0402 Multilayer Ceramic Capacitors MLCC - SMD/SMT ROHS"
-			(at 162.56 106.68 0)
+			(at 167.64 111.76 0)
 			(hide yes)
 			(show_name no)
@@
 		)
 		(property "LCSC" "C1525"
-			(at 162.56 106.68 0)
+			(at 167.64 111.76 0)
 			(hide yes)
 			(show_name no)
@@
 		)
 		(property "Stock" "20208285"
-			(at 162.56 106.68 0)
+			(at 167.64 111.76 0)
 			(hide yes)
 			(show_name no)
@@
 		)
 		(property "Price" "0.004USD"
-			(at 162.56 106.68 0)
+			(at 167.64 111.76 0)
 			(hide yes)
 			(show_name no)
@@
 		)
 		(property "Process" "SMT"
-			(at 162.56 106.68 0)
+			(at 167.64 111.76 0)
 			(hide yes)
 			(show_name no)
@@
 		)
 		(property "Minimum Qty" "20"
-			(at 162.56 106.68 0)
+			(at 167.64 111.76 0)
 			(hide yes)
 			(show_name no)
@@
 		)
 		(property "Attrition Qty" "10"
-			(at 162.56 106.68 0)
+			(at 167.64 111.76 0)
 			(hide yes)
 			(show_name no)
@@
 		)
 		(property "Class" "Basic Component"
-			(at 162.56 106.68 0)
+			(at 167.64 111.76 0)
 			(hide yes)
 			(show_name no)
@@
 		)
 		(property "Category" "Capacitors,Multilayer Ceramic Capacitors MLCC - SMD/SMT"
-			(at 162.56 106.68 0)
+			(at 167.64 111.76 0)
 			(hide yes)
 			(show_name no)
@@
 		)
 		(property "Manufacturer" "Samsung Electro-Mechanics"
-			(at 162.56 106.68 0)
+			(at 167.64 111.76 0)
 			(hide yes)
 			(show_name no)
@@
 		)
 		(property "Part" "CL05B104KO5NNNC"
-			(at 162.56 106.68 0)
+			(at 167.64 111.76 0)
 			(hide yes)
 			(show_name no)
@@
 		)
 		(property "Voltage Rated" "16V"
-			(at 164.592 110.236 0)
+			(at 166.624 109.474 90)
 			(show_name no)
 			(do_not_autoplace no)
@@
 					(size 0.8 0.8)
 				)
-				(justify left)
+				(justify right)
 			)
 		)
 		(property "Tolerance" "±10%"
-			(at 162.56 106.68 0)
+			(at 167.64 111.76 0)
 			(hide yes)
 			(show_name no)
@@
 		)
 		(property "Capacitance" "100nF"
-			(at 162.56 106.68 0)
+			(at 167.64 111.76 0)
 			(hide yes)
 			(show_name no)
@@
 		)
 		(property "Temperature Coefficient" "X7R"
-			(at 162.56 106.68 0)
+			(at 167.64 111.76 0)
 			(hide yes)
 			(show_name no)
@@
 			(project "jrdish_axis_controller"
 				(path "/10d7c3e5-be4d-4306-a59e-500b86bd141f/005a8950-9739-403f-9896-26bcf992d086"
-					(reference "C57")
+					(reference "C63")
 					(unit 1)
 				)

Commit message: Layout complete
Parts:
- added D16, D17: TPESD0402G05V, MyParts:D0402-BI, symbol MyParts:TPESD0402G05V
- added H5, H6: 210S-1*3P L=11.6MMGold-plated black, MyParts:HDR-TH_3P-P2.54-V-M-1, symbol MyParts:210S-1*3PL=11.6MMGold-platedblack
- added R55, R56: 1kΩ, PCM_JLCPCB:R_0402, symbol PCM_JLCPCB-Resistors:0402,1kΩ
Connections:
- net GND: now also D16.2 (A), D17.2 (A)
- net RS232_RX_MCU: now also R56.2
- net RS232_TX_MCU: now also R55.1
- net at CN11.1: now also H5.2; no longer U8.14 (T1OUT)
- net at CN11.2: now also H6.2; no longer U8.13 (R1IN)
- new net: D17.1 (K), H6.1, R56.1
- new net: D16.1 (K), H5.1, R55.2
- new net R1IN: H6.3, U8.13 (R1IN)
- new net T1OUT: H5.3, U8.14 (T1OUT)
Other:
- note added: "3.3V Level Rx"
- note added: "3.3V Level Tx"
- note added: "Diodes are TPESD0402G05V"
- note added: "Jumper for 3.3V vs RS232 12V"
- note added: "RS232 Level Rx"
- note added: "RS232 Level Tx"
- moved on the sheet: C62, C63, C64, C65, C66, CN10, CN11, Q3, R31, R32, U8

Commit message: Making refinements
Parts:
- added D24: TPESD0402G05V, MyParts:D0402-BI, symbol MyParts:TPESD0402G05V
- added R63: 10kΩ, PCM_JLCPCB:R_0402, symbol PCM_JLCPCB-Resistors:0402,10kΩ
Connections:
- net GND: now also D24.2 (A), R63.1
- net at CN10.1, R32.1: now also D24.1 (K)
- net at Q3.1 (G), R32.2: now also R63.2
Other:
- note added: "2N7002 is 474pF, creating a RC time constant of 4.7us. This is fast enough for this application."
- moved on the sheet: CN10, R32

Commit message: Making refinements
Connections:
- removed net GND: C63.2, C64.1, C66.1, CN10.2, CN11.3, D16.2 (A), D17.2 (A), D24.2 (A), Q3.2 (S), R63.1, U8.10 (T2IN), U8.15 (GND), U8.8 (R2IN)
- new net: CN10.2, D24.2 (A), R63.1
- new net: C64.1, C66.1
- new net: C63.2, U8.15 (GND)
Other:
- note added: "2N7002 Ciss is 20pF typ, 50pF max, creating an RC time constant of 0.2µs typ / 0.5µs max with R32. This is well within the requirements for this application."
- note removed: "2N7002 is 474pF, creating a RC time constant of 4.7us. This is fast enough for this application."
- title: (none) -> GPS 1PPS and RS232 
Changed lines of the file:
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@@
 	(generator_version "10.0")
 	(paper "A4")
+	(title_block
+		(title "GPS 1PPS and RS232 ")
+		(date "2026-04-30")
+		(rev "1.0")
+	)
 	(rectangle
 		(start 81.28 85.09)
@@
 		)
 	)
-	(text "2N7002 is 474pF, creating a RC time constant\nof 4.7us. This is fast enough for this application."
+	(text "2N7002 Ciss is 20pF typ, 50pF max, creating an RC \ntime constant of 0.2µs typ / 0.5µs max with R32. \nThis is well within the requirements for this application."
 		(exclude_from_sim no)
-		(at 86.106 72.898 0)
+		(at 81.534 73.914 0)
 		(effects
 			(font
