File: jrdish_axis_controller/power.kicad_sch (KiCad schematic)
At the start: 25 parts, among them CN6 KF2EDGR-2.54-2P, Q1 AO3407A, Q4 AO3407A, SW2 SS-12F49-G050, U4 MP2322GQH-Z

Commit message: Refinements...
Parts:
- removed CN6: KF2EDGR-2.54-2P, MyParts:CONN-TH_P2.54_KF2EDGR-2.54-2P, symbol MyParts:KF2EDGR-2.54-2P
- removed R65: 10kΩ, PCM_JLCPCB:R_0603, symbol PCM_JLCPCB-Resistors:0603,10kΩ
Connections:
- net GND: now also Q4.1 (G)
Other:
- note added: "Circuit to convert 12V DC to 3V3 DC 12V is reverse polatiry and over voltage protected MP2322 used to convert 12V to 3V3 DC 12V DC out will draw max 600mA 3V3 DC out will draw max 400mA Buck modeled after John Teel's YouTube video: https://www.youtube.com/watch?v=rLHW4gU6idU and referencing the MP2322 datasheet"
- note removed: "Circuit to convert 12V DC to 3V3 DC 12V is reverse polatiry and over voltage protected MP2322 used to convert 12V to 3V3 DC 12V DC out will draw max 600mA 3V3 DC out will draw max 400mA 12V available by a output connector: CN1 Buck modeled after John Teel's YouTube video: https://www.youtube.com/watch?v=rLHW4gU6idU and referencing the MP2322 datasheet"
- note removed: "Not to be used as 12V_IN. This is an output only."
- note removed: "Only bring out 12V to an external connector"
- note removed: "Output"
- moved on the sheet: C54
