File: jrdish_axis_controller/power.kicad_sch (KiCad schematic)
At the start: 23 parts, among them Q1 AO3407A, Q4 AO3407A, SW2 SS-12F49-G050, U4 MP2322GQH-Z

Commit message: Updates for replacing 10k resistors and encoder RC.
Parts:
- R20: LCSC C25804 -> C22356465
- R21: KiLib_Generator (none) -> SMD_2terminal_chip_molded
Changed lines of the file:
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@@
 	(title_block
 		(title "Power")
-		(date "2026-04-30")
-		(rev "1.0")
+		(date "2026-07-11")
+		(rev "1.1")
 		(company "JRSeti")
 	)
@@
 			)
 		)
+		(property "KiLib_Generator" "SMD_2terminal_chip_molded"
+			(at 223.52 118.11 0)
+			(hide yes)
+			(show_name no)
+			(do_not_autoplace no)
+			(effects
+				(font
+					(size 1.27 1.27)
+				)
+			)
+		)
 		(pin "1"
 		)
@@
 			)
 		)
-		(property "Datasheet" "https://www.lcsc.com/datasheet/lcsc_datasheet_2206010045_UNI-ROYAL-Uniroyal-Elec-0603WAF1002T5E_C25804.pdf"
+		(property "Datasheet" "https://www.lcsc.com/datasheet/lcsc_datasheet_2206010045_UNI-ROYAL-Uniroyal-Elec-0603WAF1002T5E_C22356465.pdf"
 			(at 219.71 40.64 0)
 			(hide yes)
@@
 			)
 		)
-		(property "LCSC" "C25804"
+		(property "LCSC" "C22356465"
 			(at 219.71 40.64 0)
 			(hide yes)
