File: jrdish_axis_controller/jrdish_axis_controller.kicad_pcb (KiCad board)
At the start: 4 copper layers, 100 x 100 mm, 248 parts, among them CN1 KF2EDGR-2.54-9P, CN10 KF2EDGR-2.54-2P, CN11 KF2EDGR-2.54-3P, CN12 KF2EDGR-2.54-9P, CN13 KF2EDGR-2.54-6P, CN14 KF2EDGR-2.54-6P, CN2 KF2EDGR-2.54-6P, CN3 KF2EDGR-2.54-4P, CN4 KF2EDGR-2.54-4P, CN5 KF2EDGR-2.54-4P, CN6 KF2EDGR-2.54-2P, CN7 SM04B-SRSS-TB (LF)(SN), CN8 SM04B-SRSS-TB (LF)(SN), CN9 KF2EDGR-2.54-2P, J1 Conn_ARM_SWD_TagConnect_TC2030, M1 MountingHole_2.7mm_M2.5_ISO14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, Q1 AO3407A, Q2 AO3400A, Q3 BSS138, Q4 AO3407A, Q5 BSS138, Q6 BSS138, Q7 BSS138, Q8 BSS138, SW1 DSHP04TSGER, SW2 SS-12F49-G050, U1 STM32G474RET6, U2 ISOW1432BDFMR, U3 ISOW1432BDFMR, U4 MP2322GQH-Z, U5 LTC4311ISC6#TRPBF, U6 LM75BIMX-3/NOPB, U7 W25Q32JVSSIQ_C179173, U8 SP3232EEY-L/TR, X1 7M-16.000MAAJ-T

Commit message: Refinements...
Parts:
- removed C62, C63, C64, C65, C66: 100nF, PCM_JLCPCB:C_0402
- removed CN6: KF2EDGR-2.54-2P, MyParts:CONN-TH_P2.54_KF2EDGR-2.54-2P
- removed H1, H7, H8: 210S-1*2P L=11.6MMGold-plated black, MyParts:HDR-TH_2P-P2.54-V-M-1
- removed H5, H6: 210S-1*3P L=11.6MMGold-plated black, MyParts:HDR-TH_3P-P2.54-V-M-1
- removed R1, R55, R56: 1kΩ, PCM_JLCPCB:R_0402
- removed R65: 10kΩ, PCM_JLCPCB:R_0603
- removed U8: SP3232EEY-L/TR, MyParts:TSSOP-16_L5.0-W4.4-P0.65-LS6.4-BL
- added D35: TPESD0402G05V, MyParts:D0402-BI, F.Cu at (204.4, 95.5)
- added D36: TPESD0402G05V, MyParts:D0402-BI, F.Cu at (204.4, 91.9)
- added R10: 100Ω, PCM_JLCPCB:R_0402, F.Cu at (203.3, 95.5)
- added R11: 100Ω, PCM_JLCPCB:R_0402, F.Cu at (203.3, 91.9)
- C22, C25, C26, C29: value .1uF -> 100nF
- D10, D11, D31, D32, D33, D34, D4, D5: value TPESD0402G05V -> TPESD0402G15V
- moved R20 12.0 mm to (126.5, 74.4)
- moved Q1 8.25 mm to (120.2, 75.3)
- moved Q4 7.76 mm to (120.2, 79.7)
- moved R2 7.20 mm to (153.2, 81.9), turned to -90 degrees
- moved C46 5.27 mm to (126.5, 79.4), turned to 90 degrees
- moved C47 3.85 mm to (128.8, 80.2), turned to 90 degrees
- moved F1 3.18 mm to (132.7, 81.0), turned to 180 degrees
- moved SW2 1.59 mm to (132.6, 71.4)
- moved CN11 0.49 mm to (206.4, 92.4)
- moved D32 0.05 mm to (145.7, 121.7), turned to 180 degrees
- moved D33 0.05 mm to (185.9, 121.7), turned to 0 degrees
- moved D11 0.05 mm to (183.3, 121.7), turned to 180 degrees
- turned D10 to 0 degrees
- turned D31 to 0 degrees
- turned D34 to 180 degrees
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Connections:
- D10 pad 1: 12V -> GND
- D10 pad 2: GND -> 12V
- D11 pad 1: /Axis Control - 2/LIM2_SW1_RETURN -> GND
- D11 pad 2: GND -> /Axis Control - 2/LIM2_SW1_RETURN
- D31 pad 1: 12V -> GND
- D31 pad 2: GND -> 12V
- D32 pad 1: /Axis Control - 1/LIM1_SW2_RETURN -> GND
- D32 pad 2: GND -> /Axis Control - 1/LIM1_SW2_RETURN
- D33 pad 1: 12V -> GND
- D33 pad 2: GND -> 12V
- D34 pad 1: /Axis Control - 2/LIM2_SW2_RETURN -> GND
- D34 pad 2: GND -> /Axis Control - 2/LIM2_SW2_RETURN
- D4 pad 1: 12V -> GND
- D4 pad 2: GND -> 12V
- D5 pad 1: /Axis Control - 1/LIM1_SW1_RETURN -> GND
- D5 pad 2: GND -> /Axis Control - 1/LIM1_SW1_RETURN
- Q4 pad 1: Net-(Q4-G) -> GND
Routing:
- net Net-(D35-K): track 22.0 -> 3.46 mm
- net Net-(R20-Pad2): track 19.6 -> 5.25 mm, vias 1 -> 0
- net Net-(D36-K): track 16.9 -> 3.05 mm
- net /GPS RS232/T1OUT: track 12.1 -> 0.00 mm
- net /GPS RS232/R1OUT: track 10.8 -> 0.00 mm
- net Net-(U1-PB8-BOOT0): track 12.2 -> 2.16 mm
- net 12V: track 124.1 -> 114.1 mm, vias 13 -> 14
- net /Power/12V_IN_FUSED: track 20.6 -> 10.7 mm
- net /GPS RS232/R1IN: track 9.07 -> 0.00 mm
- net /GPS RS232/T1IN: track 9.01 -> 0.00 mm, vias 2 -> 0
- net Net-(H5-Pad1): track 7.25 -> 0.00 mm
- net Net-(Q1-G): track 18.1 -> 12.6 mm
- net /Power/12V_IN: track 17.9 -> 23.4 mm
- net Net-(U8-C1-): track 3.63 -> 0.00 mm
- net RS232_RX_MCU: track 48.7 -> 52.3 mm
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Other:
- board text added: "3.3V UART Tx Rx Gnd"
- board text added: "FAN 12V DC MAX 250mA"
- board text added: "OFF"
- board text removed: "1"
- board text removed: "12V OUT 12V-Gnd"
- board text removed: "2"
- board text removed: "3"
- board text removed: "FAN 12V"
- board text removed: "RS232"
- board text removed: "RS232/3.3V Jumpers"
- board text removed: "Tx Rx Gnd"

Commit message: Minor adjustments
Parts:
- removed the C44 at (152.6, 44.0)
- removed the C45 at (183.4, 43.5)
- C13, C14: value 33pF -> 6.8pF
- X1: value 7M-16.000MAAJ-T -> NX2016SA-16MHZ-EXS00A-CS07826; footprint MyParts:OSC-SMD_4P-L3.2-W2.5-BL-OXETDLJANF-0.032768MHZ -> MyParts:CRYSTAL-SMD_4P-L2.0-W1.6-BL
- moved C13 1.58 mm to (145.9, 86.5)
- moved X1 0.77 mm to (147.8, 86.5)
- moved C14 0.45 mm to (148.0, 84.3)
Routing:
- net /RS485/RS485_2_CHASSIS: track 25.2 -> 22.7 mm
- net RS485_2_GND: track 10.4 -> 8.02 mm, vias 47 -> 52
- net /OSC_OUT: track 6.93 -> 5.42 mm
- net RS485_1_GND: vias 52 -> 54
- net GND: vias 334 -> 338
