File: jrdish_axis_controller/notes.kicad_sch (KiCad schematic)
At the start: 0 parts

Commit message: PCB layout in progress
Other:
- note added: "MCU is the STM32G474CET6, 48-pin LQFP48 package Speed and position connands are received from a host over RS485. Encoder is the E6B2-CWZ6C. Motor Controller: DM556Y. 2-Wire program/debug connector with SWO. I2C for reading I2C sensors. 2 Limit switches. USART communication to Host. 16MHz oscillator, prescalers configures for 48MHz. The STM32G474 datasheet is at https://www.st.com/resource/en/data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"
- note added: "Purpose: Control one Axis of a motor controlled system. - Modbus commands over isolated RS485. - MCU outputs motor PWM, direction, enable/disable - Input from encoder connected to motor output - Host provides configuration and position commands - MCU runs a PID loop to position/move motor - Onboard temperature sensor, MCU can turn fan on/off - I2C extender for sensors placed at the axis"
- note added: "This STM32 can be clocked up to 170MHz. It was decided to decrease this to 48MHz due to RFI concerns. The 48MHz produces much weaker harmonics above 1GHz compared to 170MHz. If speed ever becomes a concern the clock rate can be increased."
- company: (none) -> JRSeti

Commit message: Layout complete
Other:
- note added: "Purpose: Control dual axes of a motor controlled system. - Modbus commands over isolated RS485 from a host. - MCU outputs motor PWM, direction, enable/disable - Input from encoder connected to motor output - Host provides configuration and position commands - MCU runs a PID loop to position/move motors - Onboard temperature sensor, MCU can turn fan on/off - I2C extender for sensors placed at the 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"
- note removed: "Purpose: Control one Axis of a motor controlled system. - Modbus commands over isolated RS485. - MCU outputs motor PWM, direction, enable/disable - Input from encoder connected to motor output - Host provides configuration and position commands - MCU runs a PID loop to position/move motor - Onboard temperature sensor, MCU can turn fan on/off - I2C extender for sensors placed at the axis"
Changed lines of the file:
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@@
 		(company "JRSeti")
 	)
-	(text "Purpose: Control one Axis of a motor controlled\nsystem.\n\n- Modbus commands over isolated RS485.\n- MCU outputs motor PWM, direction, enable/disable\n- Input from encoder connected to motor output\n- Host provides configuration and position commands\n- MCU runs a PID loop to position/move motor\n- Onboard temperature sensor, MCU can turn fan on/off\n- I2C extender for sensors placed at the axis"
+	(text "Purpose: Control dual axes of a motor controlled\nsystem.\n\n- Modbus commands over isolated RS485 from a host.\n- MCU outputs motor PWM, direction, enable/disable\n- Input from encoder connected to motor output\n- Host provides configuration and position commands\n- MCU runs a PID loop to position/move motors\n- Onboard temperature sensor, MCU can turn fan on/off\n- I2C extender for sensors placed at the axes\n- 1PPS input from a GPS\n- NMEA sentences and 1PPS from a NEO-M9N"
 		(exclude_from_sim no)
 		(at 28.956 45.466 0)

Commit message: Making refinements
Other:
- note added: "MCU is the STM32G474CET6, 64-pin LQFP64 package Speed and position connands are received from a host over RS485. Encoder is the E6B2-CWZ6C. Motor Controller: DM556Y. 2-Wire program/debug connector with SWO. I2C for reading I2C sensors. 2 Limit switches. USART communication to Host. 16MHz oscillator, prescalers configures for 48MHz. MCU Specifications Part Number: STM32G474CET6 Package: LQFP64 Clo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"
- note removed: "MCU is the STM32G474CET6, 48-pin LQFP48 package Speed and position connands are received from a host over RS485. Encoder is the E6B2-CWZ6C. Motor Controller: DM556Y. 2-Wire program/debug connector with SWO. I2C for reading I2C sensors. 2 Limit switches. USART communication to Host. 16MHz oscillator, prescalers configures for 48MHz. The STM32G474 datasheet is at https://www.st.com/resource/en/data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"
- title: (none) -> Notes
