File: jrdish_axis_controller/fan.kicad_sch (KiCad schematic)
At the start: 7 parts, among them CN9 KF2EDGR-2.54-2P, Q2 AO3400A

Commit message: Updates for replacing 10k resistors and encoder RC.
Parts:
- R30: LCSC C25744 -> C173683
Changed lines of the file:
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@@
 	(title_block
 		(title "Fan")
-		(date "2026-04-30")
-		(rev "1.0")
+		(date "2026-07-11")
+		(rev "1.1")
 		(company "JRSeti")
 	)
@@
 			)
 		)
-		(property "Datasheet" "https://www.lcsc.com/datasheet/C15155.pdf?spm=wm.sxq.inf.ggs&lcsc_vid=FFBaV1wHQFldUVICFgBfBVJTQVJWXgBfEQRYBAFQE1YxVlNRQFdaUl1WQVlZUjtW"
+		(property "Datasheet" "https://lcsc.com/product-detail/MOSFET_AOS_AO3400A_AO3400A_C20917.html"
 			(at 143.51 109.22 0)
 			(hide yes)
@@
 			)
 		)
-		(property "Datasheet" "https://www.lcsc.com/datasheet/lcsc_datasheet_2411221126_UNI-ROYAL-Uniroyal-Elec-0402WGF1002TCE_C25744.pdf"
+		(property "Datasheet" "https://www.lcsc.com/datasheet/lcsc_datasheet_2411221126_UNI-ROYAL-Uniroyal-Elec-0402WGF1002TCE_C173683.pdf"
 			(at 128.27 99.06 0)
 			(hide yes)
@@
 			)
 		)
-		(property "LCSC" "C25744"
+		(property "LCSC" "C173683"
 			(at 128.27 99.06 0)
 			(hide yes)
